File: Modul/KiCAD/example/esp32relay/esp32relay.kicad_sch (KiCad schematic)
At the start: 0 parts

Commit message: KiCAD Sch
Parts:
- added U?: ESP32-WROOM-32, RF_Module:ESP32-WROOM-32, symbol RF_Module:ESP32-WROOM-32
Connections:
- new net: U?.1 (GND), U?.15 (GND), U?.38 (GND), U?.39 (GND)
- new net ADC2_CH4: U?.16 (IO13)
- new net ADC2_CH6: U?.13 (IO14)
- new net FLASH: U?.25 (IO0)
- new net LED: U?.24 (IO2)
- new net RELAY: U?.30 (IO18)
- new net RESET: U?.3 (EN)
- new net RX0: U?.34 (RXD0/IO3)
- new net TX0: U?.35 (TXD0/IO1)
Changed lines of the file:
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@@
 (kicad_sch (version 20211123) (generator eeschema)
   (paper "A4")
+  (global_label "LED" (shape input) (at 172.72 66.04 0) (fields_autoplaced)
+    (effects (font (size 1.27 1.27)) (justify left))
+    (property "Intersheet References" "${INTERSHEET_REFS}" (id 0) (at 178.5802 65.9606 0)
+      (effects (font (size 1.27 1.27)) (justify left) hide)
+    )
+  )
+  (global_label "TX0" (shape input) (at 172.72 63.5 0) (fields_autoplaced)
+    (effects (font (size 1.27 1.27)) (justify left))
+    (property "Intersheet References" "${INTERSHEET_REFS}" (id 0) (at 178.5198 63.4206 0)
+      (effects (font (size 1.27 1.27)) (justify left) hide)
+    )
+  )
+  (global_label "RX0" (shape input) (at 172.72 68.58 0) (fields_autoplaced)
+    (effects (font (size 1.27 1.27)) (justify left))
+    (property "Intersheet References" "${INTERSHEET_REFS}" (id 0) (at 178.8221 68.5006 0)
+      (effects (font (size 1.27 1.27)) (justify left) hide)
+    )
+  )
+  (global_label "RESET" (shape input) (at 142.24 60.96 180) (fields_autoplaced)
+    (effects (font (size 1.27 1.27)) (justify right))
+    (property "Intersheet References" "${INTERSHEET_REFS}" (id 0) (at 134.0817 60.8806 0)
+      (effects (font (size 1.27 1.27)) (justify right) hide)
+    )
+  )
+  (global_label "ADC2_CH4" (shape input) (at 172.72 78.74 0) (fields_autoplaced)
+    (effects (font (size 1.27 1.27)) (justify left))
+    (property "Intersheet References" "${INTERSHEET_REFS}" (id 0) (at 184.7488 78.6606 0)
+      (effects (font (size 1.27 1.27)) (justify left) hide)
+    )
+  )
+  (global_label "ADC2_CH6" (shape input) (at 172.72 81.28 0) (fields_autoplaced)
+    (effects (font (size 1.27 1.27)) (justify left))
+    (property "Intersheet References" "${INTERSHEET_REFS}" (id 0) (at 184.7488 81.2006 0)
+      (effects (font (size 1.27 1.27)) (justify left) hide)
+    )
+  )
+  (global_label "RELAY" (shape input) (at 172.72 91.44 0) (fields_autoplaced)
+    (effects (font (size 1.27 1.27)) (justify left))
+    (property "Intersheet References" "${INTERSHEET_REFS}" (id 0) (at 180.7574 91.3606 0)
+      (effects (font (size 1.27 1.27)) (justify left) hide)
+    )
+  )
+  (global_label "FLASH" (shape input) (at 172.72 60.96 0) (fields_autoplaced)
+    (effects (font (size 1.27 1.27)) (justify left))
+    (property "Intersheet References" "${INTERSHEET_REFS}" (id 0) (at 180.8783 60.8806 0)
+      (effects (font (size 1.27 1.27)) (justify left) hide)
+    )
+  )
+  (symbol (lib_id "RF_Module:ESP32-WROOM-32") (at 157.48 91.44 0) (unit 1)
+    (in_bom yes) (on_board yes) (fields_autoplaced)
+    (property "Reference" "U?" (id 0) (at 159.4994 53.34 0)
+      (effects (font (size 1.27 1.27)) (justify left))
+    )
+    (property "Value" "ESP32-WROOM-32" (id 1) (at 159.4994 55.88 0)
+      (effects (font (size 1.27 1.27)) (justify left))
+    )
+    (property "Footprint" "RF_Module:ESP32-WROOM-32" (id 2) (at 157.48 129.54 0)
+      (effects (font (size 1.27 1.27)) hide)
+    )
+    (property "Datasheet" "https://www.espressif.com/sites/default/files/documentation/esp32-wroom-32_datasheet_en.pdf" (id 3) (at 149.86 90.17 0)
+      (effects (font (size 1.27 1.27)) hide)
+    )
+    (pin "1")
+    (pin "10")
+    (pin "11")
+    (pin "12")
+    (pin "13")
+    (pin "14")
+    (pin "15")
+    (pin "16")
+    (pin "17")
+    (pin "18")
+    (pin "19")
+    (pin "2")
+    (pin "20")
+    (pin "21")
+    (pin "22")
+    (pin "23")
+    (pin "24")
+    (pin "25")
+    (pin "26")
+    (pin "27")
+    (pin "28")
+    (pin "29")
+    (pin "3")
+    (pin "30")
+    (pin "31")
+    (pin "32")
+    (pin "33")
+    (pin "34")
+    (pin "35")
+    (pin "36")
+    (pin "37")
+    (pin "38")
+    (pin "39")
+    (pin "4")
+    (pin "5")
+    (pin "6")
+    (pin "7")
+    (pin "8")
+    (pin "9")
+  )
   (sheet_instances
     (path "/" (page "1"))
   )
+  (symbol_instances
+    (path "/4376e9d3-2a99-4b53-a419-76ef318ac824"
+      (reference "U?") (unit 1) (value "ESP32-WROOM-32") (footprint "RF_Module:ESP32-WROOM-32")
+    )
+  )
 )

Commit message: KiCAD Sch
Parts:
- added R1, R2: 0, symbol Device:R
- gave numbers to parts that had none: 1
Connections:
- net GND: now reaches U1.1 (GND), U1.15 (GND), U1.38 (GND), U1.39 (GND)
- net GND: now also R1.2, R2.2
- net at U1.14 (IO12): now also R2.1
- net VDD: now reaches U1.2 (VDD)
- net at U1.29 (IO5): now also R1.1
Changed lines of the file:
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@@
 (kicad_sch (version 20211123) (generator eeschema)
   (paper "A4")
+  (junction (at 185.42 76.2) (diameter 0) (color 0 0 0 0)
+  )
+  (wire (pts (xy 184.15 76.2) (xy 185.42 76.2))
+    (stroke (width 0) (type default) (color 0 0 0 0))
+  )
+  (wire (pts (xy 172.72 73.66) (xy 176.53 73.66))
+    (stroke (width 0) (type default) (color 0 0 0 0))
+  )
+  (wire (pts (xy 187.96 76.2) (xy 187.96 77.47))
+    (stroke (width 0) (type default) (color 0 0 0 0))
+  )
+  (wire (pts (xy 185.42 73.66) (xy 185.42 76.2))
+    (stroke (width 0) (type default) (color 0 0 0 0))
+  )
+  (wire (pts (xy 172.72 76.2) (xy 176.53 76.2))
+    (stroke (width 0) (type default) (color 0 0 0 0))
+  )
+  (wire (pts (xy 185.42 76.2) (xy 187.96 76.2))
+    (stroke (width 0) (type default) (color 0 0 0 0))
+  )
+  (wire (pts (xy 184.15 73.66) (xy 185.42 73.66))
+    (stroke (width 0) (type default) (color 0 0 0 0))
+  )
   (global_label "LED" (shape input) (at 172.72 66.04 0) (fields_autoplaced)
     (effects (font (size 1.27 1.27)) (justify left))
@@
     )
   )
+  (symbol (lib_id "power:GND") (at 187.96 77.47 0) (unit 1)
+    (in_bom yes) (on_board yes) (fields_autoplaced)
+    (property "Reference" "#PWR03" (id 0) (at 187.96 83.82 0)
+      (effects (font (size 1.27 1.27)) hide)
+    )
+    (property "Value" "GND" (id 1) (at 187.96 82.55 0))
+    (property "Footprint" "" (id 2) (at 187.96 77.47 0)
+      (effects (font (size 1.27 1.27)) hide)
+    )
+    (property "Datasheet" "" (id 3) (at 187.96 77.47 0)
+      (effects (font (size 1.27 1.27)) hide)
+    )
+    (pin "1")
+  )
   (symbol (lib_id "RF_Module:ESP32-WROOM-32") (at 157.48 91.44 0) (unit 1)
     (in_bom yes) (on_board yes) (fields_autoplaced)
-    (property "Reference" "U?" (id 0) (at 159.4994 53.34 0)
+    (property "Reference" "U1" (id 0) (at 159.4994 53.34 0)
       (effects (font (size 1.27 1.27)) (justify left))
     )
@@
     (pin "9")
   )
+  (symbol (lib_id "power:VDD") (at 157.48 55.88 0) (unit 1)
+    (in_bom yes) (on_board yes) (fields_autoplaced)
+    (property "Reference" "#PWR01" (id 0) (at 157.48 59.69 0)
+      (effects (font (size 1.27 1.27)) hide)
+    )
+    (property "Value" "VDD" (id 1) (at 157.48 50.8 0))
+    (property "Footprint" "" (id 2) (at 157.48 55.88 0)
+      (effects (font (size 1.27 1.27)) hide)
+    )
+    (property "Datasheet" "" (id 3) (at 157.48 55.88 0)
+      (effects (font (size 1.27 1.27)) hide)
+    )
+    (pin "1")
+  )
+  (symbol (lib_id "power:GND") (at 157.48 127 0) (unit 1)
+    (in_bom yes) (on_board yes) (fields_autoplaced)
+    (property "Reference" "#PWR02" (id 0) (at 157.48 133.35 0)
+      (effects (font (size 1.27 1.27)) hide)
+    )
+    (property "Value" "GND" (id 1) (at 157.48 132.08 0))
+    (property "Footprint" "" (id 2) (at 157.48 127 0)
+      (effects (font (size 1.27 1.27)) hide)
+    )
+    (property "Datasheet" "" (id 3) (at 157.48 127 0)
+      (effects (font (size 1.27 1.27)) hide)
+    )
+    (pin "1")
+  )
+  (symbol (lib_id "Device:R") (at 180.34 76.2 90) (unit 1)
+    (in_bom yes) (on_board yes)
+    (property "Reference" "R2" (id 0) (at 187.96 74.93 90))
+    (property "Value" "0" (id 1) (at 181.61 76.2 90))
+    (property "Footprint" "" (id 2) (at 180.34 77.978 90)
+      (effects (font (size 1.27 1.27)) hide)
+    )
+    (property "Datasheet" "~" (id 3) (at 180.34 76.2 0)
+      (effects (font (size 1.27 1.27)) hide)
+    )
+    (pin "1")
+    (pin "2")
+  )
+  (symbol (lib_id "Device:R") (at 180.34 73.66 90) (unit 1)
+    (in_bom yes) (on_board yes)
+    (property "Reference" "R1" (id 0) (at 187.96 72.39 90))
+    (property "Value" "0" (id 1) (at 181.61 73.66 90))
+    (property "Footprint" "" (id 2) (at 180.34 75.438 90)
+      (effects (font (size 1.27 1.27)) hide)
+    )
+    (property "Datasheet" "~" (id 3) (at 180.34 73.66 0)
+      (effects (font (size 1.27 1.27)) hide)
+    )
+    (pin "1")
+    (pin "2")
+  )
   (sheet_instances
     (path "/" (page "1"))
   )
   (symbol_instances
+    (path "/49de18b1-99f1-447a-81ba-3d9858269671"
+      (reference "#PWR01") (unit 1) (value "VDD") (footprint "")
+    )
+    (path "/a21de203-cf1b-4201-8f30-37a22b87184b"
+      (reference "#PWR02") (unit 1) (value "GND") (footprint "")
+    )
+    (path "/224f6d9f-b061-4dfc-ad80-93148b5ab84f"
+      (reference "#PWR03") (unit 1) (value "GND") (footprint "")
+    )
+    (path "/dbf46492-5832-4a0d-bd29-77f6c79624b3"
+      (reference "R1") (unit 1) (value "0") (footprint "")
+    )
+    (path "/d91585d4-7c1e-422b-9a0c-f2f496c95b30"
+      (reference "R2") (unit 1) (value "0") (footprint "")
+    )
     (path "/4376e9d3-2a99-4b53-a419-76ef318ac824"
-      (reference "U?") (unit 1) (value "ESP32-WROOM-32") (footprint "RF_Module:ESP32-WROOM-32")
-    )
-  )
+      (reference "U1") (unit 1) (value "ESP32-WROOM-32") (footprint "RF_Module:ESP32-WROOM-32")
+    )
+  )

Commit message: KiCAD Sch
Parts:
- added C1: 100nF, symbol Device:C
- added C2: 100uF, symbol Device:C_Polarized
- added D1: LED, symbol Device:LED
- added R3, R4: 10K, symbol Device:R
- added R5: 220, symbol Device:R
- added SW1, SW2: SW_Push, symbol Switch:SW_Push
Connections:
- net FLASH: now also R4.2, SW2.1
- net GND: now also C1.2, C2.2, SW1.2, SW2.2
- net LED: now also D1.1 (K)
- net RESET: now also R3.2, SW1.1
- net VDD: now also C1.1, C2.1, R3.1, R4.1, R5.1
- new net: D1.2 (A), R5.2
- no-connect marks 0 -> 23

Commit message: KiCAD Sch
Parts:
- added R?: LDR03, OptoDevice:R_LDR_10x8.5mm_P7.6mm_Vertical, symbol Sensor_Optical:LDR03
- added RV?: R_Potentiometer_Trim, symbol Device:R_Potentiometer_Trim
Other:
- moved on the sheet: C1, C2, D1, R3, R4, R5, SW1, SW2

Commit message: KiCAD Sch
Parts:
- added D2: D, symbol Device:D
- added J1: Conn_01x03_Male, symbol Connector:Conn_01x03_Male
- added J2: Conn_01x02_Male, symbol Connector:Conn_01x02_Male
- added R7: 10K, symbol Device:R
- added U2: AMS1117-3.3, Package_TO_SOT_SMD:SOT-223-3_TabPin2, symbol Regulator_Linear:AMS1117-3.3
- gave numbers to parts that had none: 2
Connections:
- net ADC2_CH4: now also RV1.2
- net ADC2_CH6: now also R6.1, R7.2
- net GND: now also R6.2, RV1.3, J1.3 (Pin_3), J2.2 (Pin_2), U2.1 (GND)
- net RX0: now also J1.2 (Pin_2)
- net TX0: now also J1.1 (Pin_1)
- net VDD: now also RV1.1, R7.1, U2.2 (VO)
- net RELAY: no longer names the net of U1.30 (IO18)
- new net: D2.2 (A), J2.1 (Pin_1)
- new net: D2.1 (K), U2.3 (VI)
- no-connect marks 23 -> 24
Other:
- moved on the sheet: C1, C2, D1, R3, R4, R5, R6, RV1, SW1, SW2

Commit message: KiCAD Sch
Parts:
- added H1, H2, H3, H4: MountingHole, symbol Mechanical:MountingHole
Other:
- company: (none) -> PT Mencari Cinta Sejati by Achmadi ST MT
- title: (none) -> KiCAD Example 
- moved on the sheet: C1, C2, D1, D2, J1, J2, R1, R2, R3, R4, R5, R6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

Commit message: KiCAD Footprint Assigment
Parts:
- C1, C2: footprint (none) -> Capacitor_SMD:C_0805_2012Metric
- D1: footprint (none) -> LED_SMD:LED_0805_2012Metric
- D2: footprint (none) -> Diode_SMD:D_SMA
- H1, H2, H3, H4: footprint (none) -> MountingHole:MountingHole_2.5mm_Pad_Via
- J1: footprint (none) -> Connector_PinHeader_2.54mm:PinHeader_1x03_P2.54mm_Horizontal
- J2: footprint (none) -> TerminalBlock_Altech:Altech_AK300_1x02_P5.00mm_45-Degree
- R1, R2, R3, R4, R5, R7: footprint (none) -> Resistor_SMD:R_0805_2012Metric
- RV1: footprint (none) -> Potentiometer_SMD:Potentiometer_Vishay_TS53YJ_Vertical
- SW1, SW2: footprint (none) -> Button_Switch_THT:SW_PUSH_6mm
Changed lines of the file:
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@@
       (effects (font (size 1.27 1.27)) (justify right))
     )
-    (property "Footprint" "" (id 2) (at 146.05 40.64 0)
+    (property "Footprint" "LED_SMD:LED_0805_2012Metric" (id 2) (at 146.05 40.64 0)
       (effects (font (size 1.27 1.27)) hide)
     )
@@
       (effects (font (size 1.27 1.27)) (justify left))
     )
-    (property "Footprint" "" (id 2) (at 16.51 85.09 0)
+    (property "Footprint" "MountingHole:MountingHole_2.5mm_Pad_Via" (id 2) (at 16.51 85.09 0)
       (effects (font (size 1.27 1.27)) hide)
     )
@@
       (effects (font (size 1.27 1.27)) (justify right))
     )
-    (property "Footprint" "" (id 2) (at 148.59 80.01 0)
+    (property "Footprint" "Potentiometer_SMD:Potentiometer_Vishay_TS53YJ_Vertical" (id 2) (at 148.59 80.01 0)
       (effects (font (size 1.27 1.27)) hide)
     )
@@
       (effects (font (size 1.27 1.27)) (justify left))
     )
-    (property "Footprint" "" (id 2) (at 144.272 30.48 90)
+    (property "Footprint" "Resistor_SMD:R_0805_2012Metric" (id 2) (at 144.272 30.48 90)
       (effects (font (size 1.27 1.27)) hide)
     )
@@
       (effects (font (size 1.27 1.27)) (justify left))
     )
-    (property "Footprint" "" (id 2) (at 16.51 74.93 0)
+    (property "Footprint" "MountingHole:MountingHole_2.5mm_Pad_Via" (id 2) (at 16.51 74.93 0)
       (effects (font (size 1.27 1.27)) hide)
     )
@@
       (effects (font (size 1.27 1.27)) (justify left))
     )
-    (property "Footprint" "" (id 2) (at 162.2552 36.83 0)
+    (property "Footprint" "Capacitor_SMD:C_0805_2012Metric" (id 2) (at 162.2552 36.83 0)
       (effects (font (size 1.27 1.27)) hide)
     )
@@
       (effects (font (size 1.27 1.27)) (justify left))
     )
-    (property "Footprint" "" (id 2) (at 24.892 44.45 90)
+    (property "Footprint" "Resistor_SMD:R_0805_2012Metric" (id 2) (at 24.892 44.45 90)
       (effects (font (size 1.27 1.27)) hide)
     )
@@
       (effects (font (size 1.27 1.27)) (justify left))
     )
-    (property "Footprint" "" (id 2) (at 169.672 67.31 90)
+    (property "Footprint" "Resistor_SMD:R_0805_2012Metric" (id 2) (at 169.672 67.31 90)
       (effects (font (size 1.27 1.27)) hide)
     )
@@
     (property "Reference" "J2" (id 0) (at 42.545 72.39 0))
     (property "Value" "Conn_01x02_Male" (id 1) (at 42.545 74.93 0))
-    (property "Footprint" "" (id 2) (at 41.91 77.47 0)
+    (property "Footprint" "TerminalBlock_Altech:Altech_AK300_1x02_P5.00mm_45-Degree" (id 2) (at 41.91 77.47 0)
       (effects (font (size 1.27 1.27)) hide)
     )
@@
     (property "Reference" "D2" (id 0) (at 52.07 71.12 0))
     (property "Value" "D" (id 1) (at 52.07 73.66 0))
-    (property "Footprint" "" (id 2) (at 52.07 77.47 0)
+    (property "Footprint" "Diode_SMD:D_SMA" (id 2) (at 52.07 77.47 0)
       (effects (font (size 1.27 1.27)) hide)
     )
@@
     (property "Reference" "J1" (id 0) (at 57.785 30.48 0))
     (property "Value" "Conn_01x03_Male" (id 1) (at 57.785 33.02 0))
-    (property "Footprint" "" (id 2) (at 57.15 38.1 0)
+    (property "Footprint" "Connector_PinHeader_2.54mm:PinHeader_1x03_P2.54mm_Horizontal" (id 2) (at 57.15 38.1 0)
       (effects (font (size 1.27 1.27)) hide)
     )
@@
       (effects (font (size 1.27 1.27)) (justify left))
     )
-    (property "Footprint" "" (id 2) (at 16.51 69.85 0)
+    (property "Footprint" "MountingHole:MountingHole_2.5mm_Pad_Via" (id 2) (at 16.51 69.85 0)
       (effects (font (size 1.27 1.27)) hide)
     )
@@
       (effects (font (size 1.27 1.27)) (justify left))
     )
-    (property "Footprint" "" (id 2) (at 172.4152 36.83 0)
+    (property "Footprint" "Capacitor_SMD:C_0805_2012Metric" (id 2) (at 172.4152 36.83 0)
       (effects (font (size 1.27 1.27)) hide)
     )
@@
       (effects (font (size 1.27 1.27)) (justify left))
     )
-    (property "Footprint" "" (id 2) (at 24.892 25.4 90)
+    (property "Footprint" "Resistor_SMD:R_0805_2012Metric" (id 2) (at 24.892 25.4 90)
       (effects (font (size 1.27 1.27)) hide)
     )
@@
     (property "Reference" "R2" (id 0) (at 133.35 44.45 90))
     (property "Value" "0" (id 1) (at 127 45.72 90))
-    (property "Footprint" "" (id 2) (at 125.73 47.498 90)
+    (property "Footprint" "Resistor_SMD:R_0805_2012Metric" (id 2) (at 125.73 47.498 90)
       (effects (font (size 1.27 1.27)) hide)
     )
@@
     (property "Reference" "R1" (id 0) (at 133.35 41.91 90))
     (property "Value" "0" (id 1) (at 127 43.18 90))
-    (property "Footprint" "" (id 2) (at 125.73 44.958 90)
+    (property "Footprint" "Resistor_SMD:R_0805_2012Metric" (id 2) (at 125.73 44.958 90)
       (effects (font (size 1.27 1.27)) hide)
     )
@@
     (property "Reference" "SW2" (id 0) (at 39.37 41.91 0))
     (property "Value" "SW_Push" (id 1) (at 39.37 44.45 0))
-    (property "Footprint" "" (id 2) (at 39.37 44.45 0)
+    (property "Footprint" "Button_Switch_THT:SW_PUSH_6mm" (id 2) (at 39.37 44.45 0)
       (effects (font (size 1.27 1.27)) hide)
     )
@@
     (property "Reference" "SW1" (id 0) (at 39.37 24.13 0))
     (property "Value" "SW_Push" (id 1) (at 39.37 26.67 0))
-    (property "Footprint" "" (id 2) (at 39.37 26.67 0)
+    (property "Footprint" "Button_Switch_THT:SW_PUSH_6mm" (id 2) (at 39.37 26.67 0)
       (effects (font (size 1.27 1.27)) hide)
     )
@@
       (effects (font (size 1.27 1.27)) (justify left))
     )
-    (property "Footprint" "" (id 2) (at 16.51 80.01 0)
+    (property "Footprint" "MountingHole:MountingHole_2.5mm_Pad_Via" (id 2) (at 16.51 80.01 0)
       (effects (font (size 1.27 1.27)) hide)
     )
@@
     )
     (path "/4a03fd8d-7351-40da-89c3-276811b60f6c"
-      (reference "C1") (unit 1) (value "100nF") (footprint "")
+      (reference "C1") (unit 1) (value "100nF") (footprint "Capacitor_SMD:C_0805_2012Metric")
     )
     (path "/c9a3ea59-03f3-4e5f-b974-94bba4eeb410"
-      (reference "C2") (unit 1) (value "100uF") (footprint "")
+      (reference "C2") (unit 1) (value "100uF") (footprint "Capacitor_SMD:C_0805_2012Metric")
     )
     (path "/08ca79ae-1d3d-49da-9188-4200a6d96315"
-      (reference "D1") (unit 1) (value "LED") (footprint "")
+      (reference "D1") (unit 1) (value "LED") (footprint "LED_SMD:LED_0805_2012Metric")
     )
     (path "/86c3c232-c513-44d1-b2c2-ad6d48cdc8bd"
-      (reference "D2") (unit 1) (value "D") (footprint "")
+      (reference "D2") (unit 1) (value "D") (footprint "Diode_SMD:D_SMA")
     )
     (path "/bb32ba3d-3e21-4f3f-8204-e499aec217cb"
-      (reference "H1") (unit 1) (value "MountingHole") (footprint "")
+      (reference "H1") (unit 1) (value "MountingHole") (footprint "MountingHole:MountingHole_2.5mm_Pad_Via")
     )
     (path "/3bc9da20-1b84-498d-a371-dd139a1a349b"
-      (reference "H2") (unit 1) (value "MountingHole") (footprint "")
+      (reference "H2") (unit 1) (value "MountingHole") (footprint "MountingHole:MountingHole_2.5mm_Pad_Via")
     )
     (path "/f9b2aae8-f7c5-4890-8208-9244c6d31b97"
-      (reference "H3") (unit 1) (value "MountingHole") (footprint "")
+      (reference "H3") (unit 1) (value "MountingHole") (footprint "MountingHole:MountingHole_2.5mm_Pad_Via")
     )
     (path "/0950750a-20b6-41a2-b0de-a92dd2be1301"
-      (reference "H4") (unit 1) (value "MountingHole") (footprint "")
+      (reference "H4") (unit 1) (value "MountingHole") (footprint "MountingHole:MountingHole_2.5mm_Pad_Via")
     )
     (path "/b001b016-75d8-4e79-9b6f-c741feb2c038"
-      (reference "J1") (unit 1) (value "Conn_01x03_Male") (footprint "")
+      (reference "J1") (unit 1) (value "Conn_01x03_Male") (footprint "Connector_PinHeader_2.54mm:PinHeader_1x03_P2.54mm_Horizontal")
     )
     (path "/63068f0a-7295-4fd8-8d22-9f943575f98f"
-      (reference "J2") (unit 1) (value "Conn_01x02_Male") (footprint "")
+      (reference "J2") (unit 1) (value "Conn_01x02_Male") (footprint "TerminalBlock_Altech:Altech_AK300_1x02_P5.00mm_45-Degree")
     )
     (path "/dbf46492-5832-4a0d-bd29-77f6c79624b3"
-      (reference "R1") (unit 1) (value "0") (footprint "")
+      (reference "R1") (unit 1) (value "0") (footprint "Resistor_SMD:R_0805_2012Metric")
     )
     (path "/d91585d4-7c1e-422b-9a0c-f2f496c95b30"
-      (reference "R2") (unit 1) (value "0") (footprint "")
+      (reference "R2") (unit 1) (value "0") (footprint "Resistor_SMD:R_0805_2012Metric")
     )
     (path "/ca46a2e3-c402-4de8-953d-f424598095e7"
-      (reference "R3") (unit 1) (value "10K") (footprint "")
+      (reference "R3") (unit 1) (value "10K") (footprint "Resistor_SMD:R_0805_2012Metric")
     )
     (path "/4ff203d8-d747-4e5e-b3f9-172370dc9d4b"
-      (reference "R4") (unit 1) (value "10K") (footprint "")
+      (reference "R4") (unit 1) (value "10K") (footprint "Resistor_SMD:R_0805_2012Metric")
     )
     (path "/3937687f-ec32-4a2a-8367-a3d0aa3800b0"
-      (reference "R5") (unit 1) (value "220") (footprint "")
+      (reference "R5") (unit 1) (value "220") (footprint "Resistor_SMD:R_0805_2012Metric")
     )
     (path "/d2e80b94-3249-40ce-8c31-151dfee98587"
@@
     )
     (path "/588512c4-4c95-4ce2-a4f2-d94022531a13"
-      (reference "R7") (unit 1) (value "10K") (footprint "")
+      (reference "R7") (unit 1) (value "10K") (footprint "Resistor_SMD:R_0805_2012Metric")
     )
     (path "/270ec5b1-ad3d-48dc-953f-492a211115e8"
-      (reference "RV1") (unit 1) (value "R_Potentiometer_Trim") (footprint "")
+      (reference "RV1") (unit 1) (value "R_Potentiometer_Trim") (footprint "Potentiometer_SMD:Potentiometer_Vishay_TS53YJ_Vertical")
     )
     (path "/f7f5136e-6a60-41f6-a84f-3fa52bfc06fb"
-      (reference "SW1") (unit 1) (value "SW_Push") (footprint "")
+      (reference "SW1") (unit 1) (value "SW_Push") (footprint "Button_Switch_THT:SW_PUSH_6mm")
     )
     (path "/f4430897-22d3-4c1d-98b5-2d7ed72eb632"
-      (reference "SW2") (unit 1) (value "SW_Push") (footprint "")
+      (reference "SW2") (unit 1) (value "SW_Push") (footprint "Button_Switch_THT:SW_PUSH_6mm")
     )
     (path "/4376e9d3-2a99-4b53-a419-76ef318ac824"
