File: Modul/KiCAD/example/esp32relay/esp32relay.kicad_pcb (KiCad board)
At the start: 2 copper layers, 49.7 x 53.8 mm, 22 parts, among them J1 Conn_01x03_Male, J2 Conn_01x02_Male, SW1 SW_Push, SW2 SW_Push, U1 ESP32-WROOM-32, U2 AMS1117-3.3

Commit message: KiCAD PCB
Parts:
- moved C2 61.4 mm to (86.7, 45.4)
- moved R3 61.4 mm to (88.2, 48.3)
- moved U1 61.4 mm to (101.1, 53.2)
- moved C1 61.4 mm to (88.9, 45.4)
- moved D1 61.4 mm to (106.8, 65.7)
- moved H1 61.4 mm to (119.8, 73.9)
- moved H2 61.4 mm to (78.8, 73.6)
- moved H3 61.4 mm to (119.6, 39.6)
- moved J1 61.4 mm to (113.7, 47.0)
- moved R2 61.4 mm to (90.1, 62.3)
- moved R4 61.4 mm to (110.1, 65.5)
- moved R7 61.4 mm to (87.1, 60.2)
- moved SW1 61.4 mm to (88.4, 51.0)
- moved U2 61.4 mm to (104.2, 73.0)
- moved D2 61.4 mm to (104.4, 80.2)
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Routing:
- net GND: track 0.00 -> 151.0 mm, vias 0 -> 2
- net VDD: track 0.00 -> 77.1 mm, vias 0 -> 2
- net ADC2_CH6: track 0.00 -> 15.2 mm
- net FLASH: track 0.00 -> 13.6 mm
- net RESET: track 0.00 -> 13.2 mm
- net Net-(D2-Pad2): track 0.00 -> 10.7 mm
- net TX0: track 0.00 -> 5.63 mm
- net RX0: track 0.00 -> 4.40 mm
- net Net-(D2-Pad1): track 0.00 -> 4.09 mm
- net ADC2_CH4: track 0.00 -> 3.11 mm
- net Net-(R1-Pad1): track 0.00 -> 2.54 mm
- net Net-(R2-Pad1): track 0.00 -> 2.44 mm
- net LED: track 0.00 -> 2.33 mm
- net Net-(D1-Pad2): track 0.00 -> 2.28 mm
- added copper zone on B.Cu, net (none)
- added copper zone on F.Cu, net (none)
